File: Controller/hardware/main_board.sch (EAGLE design)
At the start: 43 parts, among them IC1 LINEAR_78DT, IC2 40XX_4050D, IC3 LP298XS, IC5 ATMEGA328, U1 CSTNE16M0VH3L000R0, X1 MICROSD_SMD, X4 CON-PHOENIX-508_MST2V

Commit message: working bypass capacitors
added bypass caps to the atmega328 and the 3v3 ldo per the datasheet. on the board relocated the 5v ldo bypass caps to be near the device itself.
Parts:
- added C11, C12: 0.1uF, main_board:C0.1UF_08050805
- added C13: 2.2uF, main_board:C2.2UF_08050805
- added C15: 1.0uF, main_board:C1.0UF_08050805
Connections:
- net +3V3: now also C13.2
- net GND: now also C11.1, C12.1, C13.1, C15.2
- net VCC: now also C11.2, C12.2, C15.1
Other:
- moved on the sheet: C14, C8
Changed lines of the file:
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@@
 <part name="V1" library="main_board" deviceset="GND" device=""/>
 <part name="U1" library="main_board" deviceset="CSTNE16M0VH3L000R0" device=""/>
+<part name="C11" library="main_board" deviceset="C0.1UF_0805" device="0805" value="0.1uF"/>
+<part name="C12" library="main_board" deviceset="C0.1UF_0805" device="0805" value="0.1uF"/>
+<part name="C13" library="main_board" deviceset="C2.2UF_0805" device="0805" value="2.2uF"/>
+<part name="C15" library="main_board" deviceset="C1.0UF_0805" device="0805" value="1.0uF"/>
+<part name="SUPPLY4" library="main_board" deviceset="GND" device=""/>
 </parts>
 <sheets>
@@
 <attribute name="VALUE" x="134.62" y="7.62" size="1.778" layer="96"/>
 </instance>
-<instance part="C14" gate="G$1" x="27.94" y="241.3" smashed="yes" rot="R90">
-<attribute name="NAME" x="25.019" y="240.284" size="1.778" layer="95" rot="R90"/>
-<attribute name="VALUE" x="29.464" y="241.681" size="1.778" layer="96"/>
+<instance part="C14" gate="G$1" x="35.56" y="238.76" smashed="yes" rot="R180">
+<attribute name="NAME" x="36.576" y="235.839" size="1.778" layer="95" rot="R180"/>
+<attribute name="VALUE" x="35.179" y="240.284" size="1.778" layer="96" rot="R90"/>
 </instance>
 <instance part="P+18" gate="VCC" x="48.26" y="254" smashed="yes">
@@
 <attribute name="VALUE" x="134.62" y="38.1" size="1.778" layer="96" rot="R90"/>
 </instance>
-<instance part="C8" gate="G$1" x="27.94" y="246.38" smashed="yes" rot="R90">
-<attribute name="NAME" x="25.019" y="245.364" size="1.778" layer="95" rot="R90"/>
-<attribute name="VALUE" x="29.464" y="246.761" size="1.778" layer="96"/>
+<instance part="C8" gate="G$1" x="27.94" y="243.84" smashed="yes" rot="R180">
+<attribute name="NAME" x="28.956" y="240.919" size="1.778" layer="95" rot="R180"/>
+<attribute name="VALUE" x="27.559" y="245.364" size="1.778" layer="96" rot="R90"/>
 </instance>
 <instance part="GND4" gate="1" x="66.04" y="195.58" smashed="yes">
@@
 <attribute name="NAME" x="58.42665" y="241.3133" size="1.782659375" layer="95" rot="R270"/>
 <attribute name="VALUE" x="40.6304" y="241.3101" size="1.78155" layer="96" rot="R270"/>
+</instance>
+<instance part="C11" gate="G$1" x="22.86" y="243.84" smashed="yes" rot="R180">
+<attribute name="NAME" x="23.876" y="240.919" size="1.778" layer="95" rot="R180"/>
+<attribute name="VALUE" x="22.479" y="245.364" size="1.778" layer="96" rot="R90"/>
+</instance>
+<instance part="C12" gate="G$1" x="17.78" y="243.84" smashed="yes" rot="R180">
+<attribute name="NAME" x="18.796" y="240.919" size="1.778" layer="95" rot="R180"/>
+<attribute name="VALUE" x="17.399" y="245.364" size="1.778" layer="96" rot="R90"/>
+</instance>
+<instance part="C13" gate="G$1" x="411.48" y="180.34" smashed="yes" rot="R180">
+<attribute name="NAME" x="409.956" y="177.419" size="1.778" layer="95" rot="R180"/>
+<attribute name="VALUE" x="409.956" y="182.499" size="1.778" layer="96" rot="R180"/>
+</instance>
+<instance part="C15" gate="G$1" x="370.84" y="177.8" smashed="yes">
+<attribute name="NAME" x="372.364" y="180.721" size="1.778" layer="95"/>
+<attribute name="VALUE" x="372.364" y="175.641" size="1.778" layer="96"/>
+</instance>
+<instance part="SUPPLY4" gate="1" x="411.48" y="172.72" smashed="yes">
+<attribute name="VALUE" x="411.607" y="173.101" size="1.778" layer="96"/>
 </instance>
 </instances>
@@
 <net name="GND" class="0">
 <segment>
-<wire x1="22.86" y1="241.3" x2="22.86" y2="228.6" width="0.1524" layer="91"/>
 <wire x1="22.86" y1="228.6" x2="22.86" y2="223.52" width="0.1524" layer="91"/>
-<wire x1="22.86" y1="246.38" x2="22.86" y2="241.3" width="0.1524" layer="91"/>
-<junction x="22.86" y="241.3"/>
 <pinref part="GND3" gate="1" pin="GND"/>
+<pinref part="U1" gate="G$1" pin="GND"/>
+<wire x1="43.18" y1="228.6" x2="35.56" y2="228.6" width="0.1524" layer="91"/>
+<pinref part="C12" gate="G$1" pin="1"/>
+<wire x1="35.56" y1="228.6" x2="27.94" y2="228.6" width="0.1524" layer="91"/>
+<wire x1="27.94" y1="228.6" x2="22.86" y2="228.6" width="0.1524" layer="91"/>
+<wire x1="17.78" y1="238.76" x2="17.78" y2="228.6" width="0.1524" layer="91"/>
+<wire x1="17.78" y1="228.6" x2="22.86" y2="228.6" width="0.1524" layer="91"/>
+<junction x="22.86" y="228.6"/>
+<pinref part="C11" gate="G$1" pin="1"/>
+<wire x1="22.86" y1="238.76" x2="22.86" y2="228.6" width="0.1524" layer="91"/>
+<pinref part="C8" gate="G$1" pin="1"/>
+<wire x1="27.94" y1="238.76" x2="27.94" y2="228.6" width="0.1524" layer="91"/>
+<junction x="27.94" y="228.6"/>
 <pinref part="C14" gate="G$1" pin="1"/>
-<pinref part="C8" gate="G$1" pin="1"/>
-<pinref part="U1" gate="G$1" pin="GND"/>
-<wire x1="43.18" y1="228.6" x2="22.86" y2="228.6" width="0.1524" layer="91"/>
-<junction x="22.86" y="228.6"/>
+<wire x1="35.56" y1="233.68" x2="35.56" y2="228.6" width="0.1524" layer="91"/>
+<junction x="35.56" y="228.6"/>
 </segment>
 <segment>
@@
 <wire x1="381" y1="177.8" x2="375.92" y2="177.8" width="0.1524" layer="91"/>
 <pinref part="SUPPLY1" gate="1" pin="GND"/>
-<wire x1="375.92" y1="177.8" x2="375.92" y2="167.64" width="0.1524" layer="91"/>
+<wire x1="375.92" y1="177.8" x2="375.92" y2="175.26" width="0.1524" layer="91"/>
+<pinref part="C15" gate="G$1" pin="2"/>
+<wire x1="375.92" y1="175.26" x2="375.92" y2="167.64" width="0.1524" layer="91"/>
+<wire x1="370.84" y1="175.26" x2="375.92" y2="175.26" width="0.1524" layer="91"/>
+<junction x="375.92" y="175.26"/>
 </segment>
 <segment>
@@
 <pinref part="V1" gate="1" pin="GND"/>
 <junction x="236.22" y="15.24"/>
+</segment>
+<segment>
+<pinref part="SUPPLY4" gate="1" pin="GND"/>
+<pinref part="C13" gate="G$1" pin="1"/>
 </segment>
 </net>
@@
 <wire x1="378.46" y1="182.88" x2="381" y2="182.88" width="0.1524" layer="91"/>
 <junction x="381" y="182.88"/>
+<pinref part="C15" gate="G$1" pin="1"/>
+<wire x1="370.84" y1="182.88" x2="378.46" y2="182.88" width="0.1524" layer="91"/>
+<junction x="378.46" y="182.88"/>
 </segment>
 <segment>
@@
 <wire x1="66.04" y1="248.92" x2="66.04" y2="246.38" width="0.1524" layer="91"/>
 <wire x1="66.04" y1="251.46" x2="66.04" y2="248.92" width="0.1524" layer="91"/>
-<wire x1="30.48" y1="246.38" x2="66.04" y2="246.38" width="0.1524" layer="91"/>
+<wire x1="27.94" y1="246.38" x2="66.04" y2="246.38" width="0.1524" layer="91"/>
 <junction x="66.04" y="248.92"/>
 <junction x="66.04" y="246.38"/>
@@
 <wire x1="48.26" y1="251.46" x2="66.04" y2="251.46" width="0.1524" layer="91"/>
 <junction x="66.04" y="251.46"/>
+<pinref part="C12" gate="G$1" pin="2"/>
+<pinref part="C11" gate="G$1" pin="2"/>
+<wire x1="17.78" y1="246.38" x2="22.86" y2="246.38" width="0.1524" layer="91"/>
+<wire x1="22.86" y1="246.38" x2="27.94" y2="246.38" width="0.1524" layer="91"/>
+<junction x="22.86" y="246.38"/>
+<junction x="27.94" y="246.38"/>
 </segment>
 </net>
@@
 <net name="N$20" class="0">
 <segment>
-<wire x1="66.04" y1="241.3" x2="30.48" y2="241.3" width="0.1524" layer="91"/>
+<wire x1="66.04" y1="241.3" x2="35.56" y2="241.3" width="0.1524" layer="91"/>
 <pinref part="IC5" gate="G$1" pin="AREF"/>
 <pinref part="C14" gate="G$1" pin="2"/>
@@
 <pinref part="IC3" gate="G$1" pin="VOUT"/>
 <pinref part="+3V1" gate="G$1" pin="+3V3"/>
-</segment>
-</net>
+<pinref part="C13" gate="G$1" pin="2"/>
+<wire x1="406.4" y1="182.88" x2="411.48" y2="182.88" width="0.1524" layer="91"/>
+<junction x="406.4" y="182.88"/>
+</segment>
+</net>
